Commit message: Added inertia to urdf, added inertial macros

File: description/robot.core.xacro (robot description, xacro)
@@ -1,4 +1,5 @@
 <?xml version="1.0"?>
 <robot xmlns:xacro="http://www.ros.org/wiki/xacro">
+<xacro:include filename="inertial_macros.xacro" />
 <material name="white">
     <color rgba="1 1 1 1"/>
@@ -36,4 +37,7 @@
         </geometry>
     </collision>
+    <xacro:inertial_box mass="0.5" x="0.3" y="0.3" z="0.15">
+        <origin xyz="0.15 0 0.075" rpy="0 0 0"/>
+    </xacro:inertial_box>
 </link>
 <!-- LEFT WHEEL -->
@@ -56,4 +60,7 @@
         </geometry>
     </collision>
+    <xacro:inertial_cylinder mass="0.1" length="0.05" radius="0.05">
+        <origin xyz="0 0 0" rpy="0 0 0"/>
+    </xacro:inertial_cylinder>
 </link>
 <!-- RIGHT WHEEL -->
@@ -76,4 +83,7 @@
         </geometry>
     </collision>
+    <xacro:inertial_cylinder mass="0.1" length="0.05" radius="0.05">
+        <origin xyz="0 0 0" rpy="0 0 0"/>
+    </xacro:inertial_cylinder>
 </link>
 <!-- CASTER WHEEL -->
@@ -95,4 +105,7 @@
         </geometry>
     </collision>
+        <xacro:inertial_sphere mass="0.1" radius="0.05">
+        <origin xyz="0 0 0" rpy="0 0 0"/>
+    </xacro:inertial_sphere>
 </link>
 </robot>

Commit message: Added sim env

File: description/robot.core.xacro (robot description, xacro)
@@ -41,4 +41,7 @@
     </xacro:inertial_box>
 </link>
+<gazebo reference="chassis">
+<material>Gazebo/Red</material>
+</gazebo>
 <!-- LEFT WHEEL -->
 <joint name="left_wheel_joint" type="continuous">
@@ -51,5 +54,5 @@
     <visual>
         <geometry>
-            <cylinder length="0.04" radius="0.05" />/>
+            <cylinder length="0.04" radius="0.05" />
         </geometry>
         <material name="blue"/>
@@ -57,5 +60,5 @@
      <collision>
         <geometry>
-            <cylinder length="0.04" radius="0.05" />/>
+            <cylinder length="0.04" radius="0.05" />
         </geometry>
     </collision>
@@ -64,4 +67,7 @@
     </xacro:inertial_cylinder>
 </link>
+<gazebo reference="left_wheel">
+<material>Gazebo/Black</material>
+</gazebo>
 <!-- RIGHT WHEEL -->
 <joint name="right_wheel_joint" type="continuous">
@@ -74,5 +80,5 @@
     <visual>
         <geometry>
-            <cylinder length="0.04" radius="0.05" />/>
+            <cylinder length="0.04" radius="0.05" />
         </geometry>
         <material name="blue"/>
@@ -80,5 +86,5 @@
     <collision>
         <geometry>
-            <cylinder length="0.04" radius="0.05" />/>
+            <cylinder length="0.04" radius="0.05" />
         </geometry>
     </collision>
@@ -87,4 +93,7 @@
     </xacro:inertial_cylinder>
 </link>
+<gazebo reference="right_wheel">
+<material>Gazebo/Black</material>
+</gazebo>
 <!-- CASTER WHEEL -->
 <joint name="caster_wheel_joint" type="fixed">
@@ -109,3 +118,8 @@
     </xacro:inertial_sphere>
 </link>
+<gazebo reference="caster_wheel">
+<material>Gazebo/Black</material>
+<mu1 value="0.001"/>
+<mu2 value="0.001"/>
+</gazebo>
 </robot>

File: description/robot.urdf.xacro (robot description, xacro)
@@ -2,3 +2,4 @@
 <robot xmlns:xacro="http://www.ros.org/wiki/xacro"  name="robot">
 <xacro:include filename="robot.core.xacro"/>
+<xacro:include filename="gazebo_control.xacro"/>
 </robot>
